Commit message: Add files via upload

File: my_robot.urdf (robot description, URDF)
Before this commit: robot myfirst, 1 links, 0 joints
Links:
- added link right_leg; visual box size=0.6 0.1 0.2
Joints:
- added joint base_to_right_leg: type fixed, parent base_link, child right_leg, origin xyz=0 -0.22 0.25

Commit message: Add files via upload

File: my_robot.urdf (robot description, URDF)
Before this commit: robot origins, 2 links, 1 joints
Joints:
- joint base_to_right_leg: origin xyz=0 -0.22 0.25 -> (none)
